File: content/posts/itp/spring_2020/homemade_hardware/01_letter_pcb/files/letter_i.sch (EAGLE design)
At the start: 61 parts

Commit message: hmhw 01 - new files
Connections:
- net N$3 renamed GND
- net N$4 renamed PWR
Other:
- moved on the sheet: LED1, LED10, LED11, LED12, LED13, LED14, LED15, LED16, LED17, LED18, LED19, LED2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
